File: ATMEGA32U2-DEV/HARDWARE/REV B/ATMEGA32U2 DEV.kicad_pcb (KiCad board)
At the start: 2 copper layers, 31.5 x 21.3 mm, 21 parts, among them P1 USB_A, P3 HEADER RIGHT, P4 HEADER LEFT, SW1 Push_SW, U1 ATMEGA32U2, U2 AP1117, Y1 8MHz

Commit message: Panel updates and removed AX5043
Parts:
- moved G*** 25.9 mm to (161.5, 110.4)
Other:
- rule pad_to_mask_clearance: 0 -> 0.05
- board text added: "THUNKIT ELECTRONICS"
Changed lines of the file:
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@@
     (area 128.8466 89.653147 167.5874 118.023662)
     (thickness 1.6)
-    (drawings 17)
+    (drawings 18)
     (tracks 269)
     (zones 0)
@@
     (pad_size 2.375 1.9)
     (pad_drill 0)
-    (pad_to_mask_clearance 0)
+    (pad_to_mask_clearance 0.05)
     (aux_axis_origin 0 0)
     (visible_elements FFFEFFFF)
@@
   )
   (module MOD:lightning (layer B.Cu)
-    (at 135.636 108.966 270)
+    (at 161.544 110.363 270)
     (fp_text reference G*** (at 0 0 270) (layer B.SilkS) hide
       (effects (font (thickness 0.3)) (justify mirror))
@@
       (xy 0.31437 1.300123) (xy 0.314354 1.28972)) (layer B.SilkS) (width 0.01))
   )
+  (gr_text "THUNKIT ELECTRONICS" (at 162.687 97.028 90) (layer B.SilkS)
+    (effects (font (size 0.75 0.75) (thickness 0.15)) (justify left mirror))
+  )
   (gr_line (start 133.096 114.7445) (end 135.636 114.7445) (layer Edge.Cuts) (width 0.1))
